Commit message: controller state broadcaster working

File: mars_rover/urdf/curiosity_mars_rover.xacro (robot description, xacro)
@@ -22,3 +22,21 @@
 	<xacro:arm/>
 	<xacro:sensor_mast/>
+    <ros2_control name="IgnitionSystem" type="system">
+        <hardware>
+            <plugin>ign_ros2_control/IgnitionSystem</plugin>
+        </hardware>
+        <joint name="arm_01_joint">
+            <command_interface name="position">
+            </command_interface>
+            <state_interface name="position" />
+            <state_interface name="velocity" />
+        </joint>
+    </ros2_control>
+    <gazebo>
+        <plugin filename="libign_ros2_control-system" name="ign_ros2_control::IgnitionROS2ControlPlugin">
+        <robot_param>robot_description</robot_param>
+        <robot_param_node>robot_state_publisher</robot_param_node>
+        <parameters>$(find mars_rover)/config/mars_rover_control.yaml</parameters>
+        </plugin>
+    </gazebo>
 </robot>

Commit message: control arm

File: mars_rover/urdf/curiosity_mars_rover.xacro (robot description, xacro)
@@ -32,4 +32,28 @@
             <state_interface name="velocity" />
         </joint>
+        <joint name="arm_02_joint">
+            <command_interface name="position">
+            </command_interface>
+            <state_interface name="position" />
+            <state_interface name="velocity" />
+        </joint>
+        <joint name="arm_03_joint">
+            <command_interface name="position">
+            </command_interface>
+            <state_interface name="position" />
+            <state_interface name="velocity" />
+        </joint>
+        <joint name="arm_04_joint">
+            <command_interface name="position">
+            </command_interface>
+            <state_interface name="position" />
+            <state_interface name="velocity" />
+        </joint>
+        <joint name="arm_tools_joint">
+            <command_interface name="position">
+            </command_interface>
+            <state_interface name="position" />
+            <state_interface name="velocity" />
+        </joint>
     </ros2_control>
     <gazebo>

Commit message: added wheel velocity and mast position control

File: mars_rover/urdf/curiosity_mars_rover.xacro (robot description, xacro)
@@ -27,30 +27,70 @@
         </hardware>
         <joint name="arm_01_joint">
-            <command_interface name="position">
-            </command_interface>
+            <command_interface name="position" />
             <state_interface name="position" />
             <state_interface name="velocity" />
         </joint>
         <joint name="arm_02_joint">
-            <command_interface name="position">
-            </command_interface>
+            <command_interface name="position" />
             <state_interface name="position" />
             <state_interface name="velocity" />
         </joint>
         <joint name="arm_03_joint">
-            <command_interface name="position">
-            </command_interface>
+            <command_interface name="position" />
             <state_interface name="position" />
             <state_interface name="velocity" />
         </joint>
         <joint name="arm_04_joint">
-            <command_interface name="position">
-            </command_interface>
+            <command_interface name="position" />
             <state_interface name="position" />
             <state_interface name="velocity" />
         </joint>
         <joint name="arm_tools_joint">
-            <command_interface name="position">
-            </command_interface>
+            <command_interface name="position" />
+            <state_interface name="position" />
+            <state_interface name="velocity" />
+        </joint>
+        <joint name="mast_p_joint">
+            <command_interface name="position" />
+            <state_interface name="position" />
+            <state_interface name="velocity" />
+        </joint>
+        <joint name="mast_02_joint">
+            <command_interface name="position" />
+            <state_interface name="position" />
+            <state_interface name="velocity" />
+        </joint>
+        <joint name="mast_cameras_joint">
+            <command_interface name="position" />
+            <state_interface name="position" />
+            <state_interface name="velocity" />
+        </joint>
+        <joint name="front_wheel_L_joint">
+            <command_interface name="velocity" />
+            <state_interface name="position" />
+            <state_interface name="velocity" />
+        </joint>
+        <joint name="middle_wheel_L_joint">
+            <command_interface name="velocity" />
+            <state_interface name="position" />
+            <state_interface name="velocity" />
+        </joint>
+        <joint name="back_wheel_L_joint">
+            <command_interface name="velocity" />
+            <state_interface name="position" />
+            <state_interface name="velocity" />
+        </joint>
+        <joint name="front_wheel_R_joint">
+            <command_interface name="velocity" />
+            <state_interface name="position" />
+            <state_interface name="velocity" />
+        </joint>
+        <joint name="middle_wheel_R_joint">
+            <command_interface name="velocity" />
+            <state_interface name="position" />
+            <state_interface name="velocity" />
+        </joint>
+        <joint name="back_wheel_R_joint">
+            <command_interface name="velocity" />
             <state_interface name="position" />
             <state_interface name="velocity" />

Commit message: all controllers launch correctly

File: mars_rover/urdf/curiosity_mars_rover.xacro (robot description, xacro)
@@ -96,4 +96,48 @@
             <state_interface name="velocity" />
         </joint>
+        <joint name="suspension_steer_F_L_joint">
+            <command_interface name="position" />
+            <state_interface name="position" />
+            <state_interface name="velocity" />
+        </joint>
+        <joint name="suspension_steer_B_L_joint">
+            <command_interface name="position" />
+            <state_interface name="position" />
+            <state_interface name="velocity" />
+        </joint>
+        <joint name="suspension_steer_F_R_joint">
+            <command_interface name="position" />
+            <state_interface name="position" />
+            <state_interface name="velocity" />
+        </joint>
+        <joint name="suspension_steer_B_R_joint">
+            <command_interface name="position" />
+            <state_interface name="position" />
+            <state_interface name="velocity" />
+        </joint>
+        <joint name="suspension_arm_F_L_joint">
+            <command_interface name="position" />
+            <state_interface name="position" />
+        </joint>
+        <joint name="suspension_arm_B_L_joint">
+            <command_interface name="position" />
+            <state_interface name="position" />
+        </joint>
+        <joint name="suspension_arm_B2_L_joint">
+            <command_interface name="position" />
+            <state_interface name="position" />
+        </joint>
+        <joint name="suspension_arm_F_R_joint">
+            <command_interface name="position" />
+            <state_interface name="position" />
+        </joint>
+        <joint name="suspension_arm_B_R_joint">
+            <command_interface name="position" />
+            <state_interface name="position" />
+        </joint>
+        <joint name="suspension_arm_B2_R_joint">
+            <command_interface name="position" />
+            <state_interface name="position" />
+        </joint>
     </ros2_control>
     <gazebo>

Commit message: added arm service and bring up camera

File: mars_rover/urdf/curiosity_mars_rover.xacro (robot description, xacro)
@@ -137,3 +137,34 @@
         </plugin>
     </gazebo>
+    <gazebo reference="camera_link">
+        <sensor type="camera" name="camera_sensor">
+            <visualize>1</visualize>
+            <update_rate>10.0</update_rate>
+            <camera>
+                <pose>1.0 0 0 0 0 -1.57</pose>
+                <horizontal_fov>1.3962634</horizontal_fov>
+                <image>
+                    <width>800</width>
+                    <height>800</height>
+                    <format>R8G8B8</format>
+                </image>
+                <clip>
+                <near>0.01</near>
+                <far>100</far>
+                </clip>
+                <noise>
+                <type>gaussian</type>
+                <stddev>0.007</stddev>
+                </noise>
+            </camera>
+            <always_on>1</always_on>
+            <topic>image_raw</topic>
+            <plugin
+                filename="ignition-gazebo-sensors-system"
+                name="ignition::gazebo::systems::Sensors">
+                <render_engine>ogre2</render_engine>
+                <background_color>1 1 1 1</background_color>
+            </plugin>
+        </sensor>
+    </gazebo>
 </robot>

File: mars_rover/urdf/sensor_mast.xacro (robot description, xacro)
@@ -230,5 +230,5 @@
         <parent link="mast_cameras"/>
         <child link="camera_link"/>
-        <origin xyz="0.13642 -0.218683 0.222314" rpy="0 0 ${PI}"/>
+        <origin xyz="0.13642 -0.218683 0.222314" rpy="0 0 ${-PI/2}"/>
     </joint>
   </xacro:macro>

Commit message: reorg control plugin in urdf

File: mars_rover/urdf/curiosity_mars_rover.xacro (robot description, xacro)
@@ -22,165 +22,3 @@
 	<xacro:arm/>
 	<xacro:sensor_mast/>
-    <ros2_control name="IgnitionSystem" type="system">
-        <hardware>
-            <plugin>ign_ros2_control/IgnitionSystem</plugin>
-        </hardware>
-        <!-- Arm Joints Interfaces-->
-        <joint name="arm_01_joint">
-            <command_interface name="position" />
-            <state_interface name="position" />
-            <state_interface name="velocity" />
-        </joint>
-        <joint name="arm_02_joint">
-            <command_interface name="position" />
-            <state_interface name="position" />
-            <state_interface name="velocity" />
-        </joint>
-        <joint name="arm_03_joint">
-            <command_interface name="position" />
-            <state_interface name="position" />
-            <state_interface name="velocity" />
-        </joint>
-        <joint name="arm_04_joint">
-            <command_interface name="position" />
-            <state_interface name="position" />
-            <state_interface name="velocity" />
-        </joint>
-        <joint name="arm_tools_joint">
-            <command_interface name="position" />
-            <state_interface name="position" />
-            <state_interface name="velocity" />
-        </joint>
-        <!-- Mast Joints Interfaces-->
-        <joint name="mast_p_joint">
-            <command_interface name="position" />
-            <state_interface name="position" />
-            <state_interface name="velocity" />
-        </joint>
-        <joint name="mast_02_joint">
-            <command_interface name="position" />
-            <state_interface name="position" />
-            <state_interface name="velocity" />
-        </joint>
-        <joint name="mast_cameras_joint">
-            <command_interface name="position" />
-            <state_interface name="position" />
-            <state_interface name="velocity" />
-        </joint>
-        <!-- Wheel Joints Interfaces-->
-        <joint name="front_wheel_L_joint">
-            <command_interface name="velocity" />
-        </joint>
-        <joint name="middle_wheel_L_joint">
-            <command_interface name="velocity" />
-        </joint>
-        <joint name="back_wheel_L_joint">
-            <command_interface name="velocity" />
-        </joint>
-        <joint name="front_wheel_R_joint">
-            <command_interface name="velocity" />
-        </joint>
-        <joint name="middle_wheel_R_joint">
-            <command_interface name="velocity" />
-        </joint>
-        <joint name="back_wheel_R_joint">
-            <command_interface name="velocity" />
-        </joint>
-        <!-- Steering Joints Interfaces-->
-        <joint name="suspension_steer_F_L_joint">
-            <command_interface name="position" />
-            <state_interface name="position" />
-            <state_interface name="velocity" />
-        </joint>
-        <joint name="suspension_steer_B_L_joint">
-            <command_interface name="position" />
-            <state_interface name="position" />
-            <state_interface name="velocity" />
-        </joint>
-        <joint name="suspension_steer_F_R_joint">
-            <command_interface name="position" />
-            <state_interface name="position" />
-            <state_interface name="velocity" />
-        </joint>
-        <joint name="suspension_steer_B_R_joint">
-            <command_interface name="position" />
-            <state_interface name="position" />
-            <state_interface name="velocity" />
-        </joint>
-        <!-- Suspension Arms Interfaces-->
-        <joint name="suspension_arm_F_L_joint">
-            <command_interface name="effort"/>
-            <state_interface name="position"/>
-            <state_interface name="velocity"/>
-            <state_interface name="effort"/>
-        </joint>
-        <joint name="suspension_arm_B_L_joint">
-            <command_interface name="effort"/>
-            <state_interface name="position"/>
-            <state_interface name="velocity"/>
-            <state_interface name="effort"/>
-        </joint>
-        <joint name="suspension_arm_B2_L_joint">
-            <command_interface name="effort"/>
-            <state_interface name="position"/>
-            <state_interface name="velocity"/>
-            <state_interface name="effort"/>
-        </joint>
-        <joint name="suspension_arm_F_R_joint">
-            <command_interface name="effort"/>
-            <state_interface name="position"/>
-            <state_interface name="velocity"/>
-            <state_interface name="effort"/>
-        </joint>
-        <joint name="suspension_arm_B_R_joint">
-            <command_interface name="effort"/>
-            <state_interface name="position"/>
-            <state_interface name="velocity"/>
-            <state_interface name="effort"/>
-        </joint>
-        <joint name="suspension_arm_B2_R_joint">
-            <command_interface name="effort"/>
-            <state_interface name="position"/>
-            <state_interface name="velocity"/>
-            <state_interface name="effort"/>
-        </joint>
-    </ros2_control>
-    <gazebo>
-        <plugin filename="libign_ros2_control-system" name="ign_ros2_control::IgnitionROS2ControlPlugin">
-        <robot_param>robot_description</robot_param>
-        <robot_param_node>robot_state_publisher</robot_param_node>
-        <parameters>$(find mars_rover)/config/mars_rover_control.yaml</parameters>
-        </plugin>
-    </gazebo>
-    <gazebo reference="camera_link">
-        <sensor type="camera" name="camera_sensor">
-            <visualize>1</visualize>
-            <update_rate>10.0</update_rate>
-            <camera>
-                <pose>1.0 0 0 0 0 -1.57</pose>
-                <horizontal_fov>1.3962634</horizontal_fov>
-                <image>
-                    <width>800</width>
-                    <height>800</height>
-                    <format>R8G8B8</format>
-                </image>
-                <clip>
-                <near>0.01</near>
-                <far>100</far>
-                </clip>
-                <noise>
-                <type>gaussian</type>
-                <stddev>0.007</stddev>
-                </noise>
-            </camera>
-            <always_on>1</always_on>
-            <topic>image_raw</topic>
-            <plugin
-                filename="ignition-gazebo-sensors-system"
-                name="ignition::gazebo::systems::Sensors">
-                <render_engine>ogre2</render_engine>
-                <background_color>0.9 0.753 0.66 1</background_color>
-            </plugin>
-        </sensor>
-    </gazebo>
 </robot>
