Commit message: suspension arm working with terrain

File: mars_rover/urdf/arm.xacro (robot description, xacro)
@@ -58,5 +58,5 @@
 		<limit lower="${-arm_01_limit}" upper="${arm_01_limit}" effort="10000.0" velocity="100.0"/>
         <axis xyz="0 0 1"/>
-        <joint_properties damping="0.0" friction="0.0"/>
+        <dynamics damping="0.0" friction="0.0"/>
 	</joint>
     <transmission name="arm_01_trans">
@@ -126,5 +126,5 @@
 		<limit lower="${-arm_02_limit}" upper="${arm_02_limit}" effort="10000.0" velocity="100.0"/>
         <axis xyz="1 0 0"/>
-        <joint_properties damping="0.0" friction="0.0"/>
+        <dynamics damping="0.0" friction="0.0"/>
 	</joint>
     <transmission name="arm_02_trans">
@@ -194,5 +194,5 @@
 		<limit lower="${-arm_03_limit}" upper="${arm_03_limit}" effort="10000.0" velocity="100.0"/>
         <axis xyz="1 0 0"/>
-        <joint_properties damping="0.0" friction="0.0"/>
+        <dynamics damping="0.0" friction="0.0"/>
 	</joint>
     <transmission name="arm_03_trans">
@@ -262,5 +262,5 @@
 		<limit lower="${-arm_04_limit}" upper="${arm_04_limit}" effort="10000.0" velocity="100.0"/>
         <axis xyz="0 1 0"/>
-        <joint_properties damping="0.0" friction="0.0"/>
+        <dynamics damping="0.0" friction="0.0"/>
 	</joint>
     <transmission name="arm_04_trans">
@@ -330,5 +330,5 @@
 		<limit effort="10000.0" velocity="100.0"/>
         <axis xyz="0 0 1"/>
-        <joint_properties damping="0.0" friction="0.0"/>
+        <dynamics damping="0.0" friction="0.0"/>
 	</joint>
     <transmission name="arm_tools_trans">

File: mars_rover/urdf/curiosity_mars_rover.xacro (robot description, xacro)
@@ -6,5 +6,5 @@
 	<xacro:include filename="$(find mars_rover)/urdf/curiosity_mars_rover_properties.xacro" />
 	<!-- Gazebo aspects of the robot -->
-	<!-- <xacro:include filename="$(find mars_rover)/urdf/curiosity_mars_rover.gazebo" /> -->
+	<xacro:include filename="$(find mars_rover)/urdf/curiosity_mars_rover.gazebo" />
 	<!-- Chasis -->
 	<xacro:include filename="$(find mars_rover)/urdf/chassis.xacro" />

File: mars_rover/urdf/curiosity_mars_rover.xacro.urdf (robot description, URDF)
Before this commit: robot curiosity_mars_rover, 49 links, 48 joints
Joints:
- joint suspension_arm_B2_L_joint: limit lower=-1.2 upper=0.1 effort=10000.0 velocity=10.0 -> lower=-1.2 upper=1.2 effort=10000.0 velocity=10.0
- joint suspension_arm_B2_R_joint: limit lower=-1.2 upper=0.1 effort=10000.0 velocity=10.0 -> lower=-1.2 upper=1.2 effort=10000.0 velocity=10.0

File: mars_rover/urdf/curiosity_mars_rover_properties.xacro (robot description, xacro)
@@ -32,5 +32,5 @@
 	<xacro:property name="suspension_arm_B2_L_Z" value="0.631338"/>
 	<xacro:property name="suspension_arm_B2_lower_limit" value="-1.2"/>
-	<xacro:property name="suspension_arm_B2_upper_limit" value="0.1"/>
+	<xacro:property name="suspension_arm_B2_upper_limit" value="1.2"/>
 	<xacro:property name="suspension_steer_F_L_Mass" value="${TreeMass/TreeParts}"/>
 	<xacro:property name="suspension_steer_F_L_X" value="0.528399"/>
@@ -46,6 +46,6 @@
 	<xacro:property name="suspension_effort" value="10000.0"/>
 	<xacro:property name="suspension_speed" value="10.0"/>
-	<xacro:property name="suspension_damping" value="0.5"/>
-	<xacro:property name="suspension_friction" value="0.5"/>
+	<xacro:property name="suspension_damping" value="0.0"/>
+	<xacro:property name="suspension_friction" value="0.0"/>
 	<!-- Wheels properties -->
 	<xacro:property name="wheelWidth" value="0.39473"/>

File: mars_rover/urdf/left_wheel_group.xacro (robot description, xacro)
@@ -65,5 +65,5 @@
 		<limit lower="${-suspension_arm_F_L_limit}" upper="${suspension_arm_F_L_limit}" effort="${suspension_effort}" velocity="${suspension_speed}"/>
         <axis xyz="1 0 0"/>
-		<joint_properties damping="${suspension_damping}" friction="${suspension_friction}"/>
+		<dynamics damping="${suspension_damping}" friction="${suspension_friction}"/>
 	</joint>
 	<transmission name="suspension_arm_F_L_trans">
@@ -109,5 +109,5 @@
 		<limit lower="${-suspension_arm_B_L_limit}" upper="${suspension_arm_B_L_limit}" effort="${suspension_effort}" velocity="${suspension_speed}"/>
         <axis xyz="1 0 0"/>
-		<joint_properties damping="${suspension_damping}" friction="${suspension_friction}"/>
+		<dynamics damping="${suspension_damping}" friction="${suspension_friction}"/>
 	</joint>
 	<transmission name="suspension_arm_B_L_trans">
@@ -177,5 +177,5 @@
 		<limit lower="${suspension_arm_B2_lower_limit}" upper="${suspension_arm_B2_upper_limit}" effort="${suspension_effort}" velocity="${suspension_speed}"/>
         <axis xyz="1 0 0"/>
-		<joint_properties damping="${suspension_damping}" friction="${suspension_friction}"/>
+		<dynamics damping="${suspension_damping}" friction="${suspension_friction}"/>
 	</joint>
 	<transmission name="suspension_arm_B2_L_trans">

File: mars_rover/urdf/right_wheel_group.xacro (robot description, xacro)
@@ -65,5 +65,5 @@
 		<limit lower="${-suspension_arm_F_L_limit}" upper="${suspension_arm_F_L_limit}" effort="${suspension_effort}" velocity="${suspension_speed}"/>
         <axis xyz="1 0 0"/>
-		<joint_properties damping="${suspension_damping}" friction="${suspension_friction}"/>
+		<dynamics damping="${suspension_damping}" friction="${suspension_friction}"/>
 	</joint>
   	<transmission name="suspension_arm_F_R_trans">
@@ -109,5 +109,5 @@
 		<limit lower="${-suspension_arm_B_L_limit}" upper="${suspension_arm_B_L_limit}" effort="${suspension_effort}" velocity="${suspension_speed}"/>
         <axis xyz="1 0 0"/>
-		<joint_properties damping="${suspension_damping}" friction="${suspension_friction}"/>
+		<dynamics damping="${suspension_damping}" friction="${suspension_friction}"/>
 	</joint>
   	<transmission name="suspension_arm_B_R_trans">
@@ -177,5 +177,5 @@
 		<limit lower="${suspension_arm_B2_lower_limit}" upper="${suspension_arm_B2_upper_limit}" effort="${suspension_effort}" velocity="${suspension_speed}"/>
         <axis xyz="1 0 0"/>
-		<joint_properties damping="${suspension_damping}" friction="${suspension_friction}"/>
+		<dynamics damping="${suspension_damping}" friction="${suspension_friction}"/>
 	</joint>
   	<transmission name="suspension_arm_B2_R_trans">

File: mars_rover/urdf/sensor_mast.xacro (robot description, xacro)
@@ -58,5 +58,5 @@
 		<limit lower="${mast_p_lower_limit}" upper="${mast_p_upper_limit}" effort="10000.0" velocity="100.0"/>
         <axis xyz="0 1 0"/>
-        <joint_properties damping="0.0" friction="0.0"/>
+        <dynamics damping="0.0" friction="0.0"/>
 	</joint>
     <transmission name="mast_p_trans">
@@ -126,5 +126,5 @@
 		<limit effort="10000.0" velocity="100.0"/>
         <axis xyz="0 0 1"/>
-        <joint_properties damping="0.0" friction="0.0"/>
+        <dynamics damping="0.0" friction="0.0"/>
 	</joint>
     <transmission name="mast_02_trans">
@@ -194,5 +194,5 @@
 		<limit lower="${-mast_cameras_limit}" upper="${mast_cameras_limit}" effort="10000.0" velocity="100.0"/>
         <axis xyz="1 0 0"/>
-        <joint_properties damping="0.0" friction="0.0"/>
+        <dynamics damping="0.0" friction="0.0"/>
 	</joint>
     <transmission name="mast_02_trans">

File: mars_rover/urdf/wheel.xacro (robot description, xacro)
@@ -44,5 +44,5 @@
 		<limit effort="10000.0" velocity="100.0"/>
         <axis xyz="1 0 0"/>
-        <joint_properties damping="0.0" friction="0.0"/>
+        <dynamics damping="0.0" friction="0.0"/>
 	</joint>
     <transmission name="${wheel_name}_trans">
