Commit message: fix steering wheel bug

File: mars_rover/urdf/curiosity_mars_rover.xacro.urdf (robot description, URDF)
Before this commit: robot curiosity_mars_rover, 49 links, 48 joints
Joints:
- joint arm_03_joint: limit lower=-1.57 upper=1.57 effort=10000.0 velocity=100.0 -> lower=-5.0 upper=5.0 effort=10000.0 velocity=100.0

File: mars_rover/urdf/curiosity_mars_rover_properties.xacro (robot description, xacro)
@@ -46,6 +46,6 @@
 	<xacro:property name="suspension_effort" value="10000.0"/>
 	<xacro:property name="suspension_speed" value="10.0"/>
-	<xacro:property name="suspension_damping" value="0.0"/>
-	<xacro:property name="suspension_friction" value="0.0"/>
+	<xacro:property name="suspension_damping" value="0.5"/>
+	<xacro:property name="suspension_friction" value="0.5"/>
 	<!-- Wheels properties -->
 	<xacro:property name="wheelWidth" value="0.39473"/>
@@ -69,5 +69,5 @@
 	<xacro:property name="arm_03_Y" value="0.178607"/>
 	<xacro:property name="arm_03_Z" value="0.878958"/>
-	<xacro:property name="arm_03_limit" value="1.57"/>
+	<xacro:property name="arm_03_limit" value="5.0"/>
 	<xacro:property name="arm_04_Mass" value="${armMass/armParts}"/>
 	<xacro:property name="arm_04_X" value="0.32452"/>

Commit message: fixing demo with old structure
Signed-off-by: Dharini Dutia <dharini@openrobotics.org>

File: mars_rover/urdf/curiosity_mars_rover.xacro.urdf (robot description, URDF)
Before this commit: robot curiosity_mars_rover, 49 links, 48 joints
Links:
- link chassis: geometry collision mesh filename=package://meshes/chassis_full_fixed_glitch_v2.dae scale=1.0 1.0 1.0; visual mesh filename=package://meshes/chassis_full_fixed_glitch_v2.dae scale=1.0 1.0 1.0
