Commit message: using relative paths in urdf
Signed-off-by: tonylitianyu <tonylitianyu@gmail.com>

File: canadarm/urdf/SSRMS_Canadarm2.urdf (robot description, URDF)
Before this commit: robot SSRMS_Canadarm2, 9 links, 8 joints
Links:
- link B1: geometry visual mesh filename=package://sdf/meshes/joint_v3_0.dae scale=1.0 1.0 1.0
- link B2: geometry visual mesh filename=package://sdf/meshes/joint_v3_0.dae scale=1.0 1.0 1.0
- link B3: geometry visual cylinder length=0.5 radius=0.165; visual mesh filename=package://sdf/meshes/joint_v3_0.dae scale=1.0 1.0 1.0
- link B4: geometry visual mesh filename=package://sdf/meshes/joint_v3_0.dae scale=1.0 1.0 1.0; visual mesh filename=package://sdf/meshes/link_joint_v2_1.dae scale=1.0 1.0 1.0
- link B5: geometry visual mesh filename=package://sdf/meshes/joint_v3_0.dae scale=1.0 1.0 1.0
- link B6: geometry visual mesh filename=package://sdf/meshes/joint_v3_0.dae scale=1.0 1.0 1.0
- link Base_SSRMS: geometry visual mesh filename=package://sdf/meshes/ee.dae scale=1.0 1.0 1.0
- link EE_SSRMS: geometry visual mesh filename=package://sdf/meshes/ee.dae scale=1.0 1.0 1.0

File: mars_rover/urdf/arm.xacro (robot description, xacro)
@@ -31,12 +31,12 @@
 					rpy="0 0 0"/>
 			<geometry>
-				<mesh filename="/home/spaceros-user/src/spaceros_demo/install/mars_rover/share/mars_rover/meshes/arm_01_fixed.dae" scale="${scale_XYZ} ${scale_XYZ} ${scale_XYZ}"/>
-			</geometry>
-		</collision>
-		<visual>
-			<origin xyz="0 0 0"
-					rpy="0 0 0"/>
-			<geometry>
-				<mesh filename="/home/spaceros-user/src/spaceros_demo/install/mars_rover/share/mars_rover/meshes/arm_01_fixed.dae" scale="${scale_XYZ} ${scale_XYZ} ${scale_XYZ}"/>
+				<mesh filename="package://mars_rover/meshes/arm_01_fixed.dae" scale="${scale_XYZ} ${scale_XYZ} ${scale_XYZ}"/>
+			</geometry>
+		</collision>
+		<visual>
+			<origin xyz="0 0 0"
+					rpy="0 0 0"/>
+			<geometry>
+				<mesh filename="package://mars_rover/meshes/arm_01_fixed.dae" scale="${scale_XYZ} ${scale_XYZ} ${scale_XYZ}"/>
 			</geometry>
 		</visual>
@@ -99,12 +99,12 @@
 					rpy="0 0 0"/>
 			<geometry>
-				<mesh filename="/home/spaceros-user/src/spaceros_demo/install/mars_rover/share/mars_rover/meshes/arm_01_fixed.dae" scale="${scale_XYZ} ${scale_XYZ} ${scale_XYZ}"/>
-			</geometry>
-		</collision>
-		<visual>
-			<origin xyz="0 0 0"
-					rpy="0 0 0"/>
-			<geometry>
-				<mesh filename="/home/spaceros-user/src/spaceros_demo/install/mars_rover/share/mars_rover/meshes/arm_02_fixed.dae" scale="${scale_XYZ} ${scale_XYZ} ${scale_XYZ}"/>
+				<mesh filename="package://mars_rover/meshes/arm_01_fixed.dae" scale="${scale_XYZ} ${scale_XYZ} ${scale_XYZ}"/>
+			</geometry>
+		</collision>
+		<visual>
+			<origin xyz="0 0 0"
+					rpy="0 0 0"/>
+			<geometry>
+				<mesh filename="package://mars_rover/meshes/arm_02_fixed.dae" scale="${scale_XYZ} ${scale_XYZ} ${scale_XYZ}"/>
 			</geometry>
 		</visual>
@@ -167,12 +167,12 @@
 					rpy="0 0 0"/>
 			<geometry>
-				<mesh filename="/home/spaceros-user/src/spaceros_demo/install/mars_rover/share/mars_rover/meshes/arm_03_fixed.dae" scale="${scale_XYZ} ${scale_XYZ} ${scale_XYZ}"/>
-			</geometry>
-		</collision>
-		<visual>
-			<origin xyz="0 0 0"
-					rpy="0 0 0"/>
-			<geometry>
-				<mesh filename="/home/spaceros-user/src/spaceros_demo/install/mars_rover/share/mars_rover/meshes/arm_03_fixed.dae" scale="${scale_XYZ} ${scale_XYZ} ${scale_XYZ}"/>
+				<mesh filename="package://mars_rover/meshes/arm_03_fixed.dae" scale="${scale_XYZ} ${scale_XYZ} ${scale_XYZ}"/>
+			</geometry>
+		</collision>
+		<visual>
+			<origin xyz="0 0 0"
+					rpy="0 0 0"/>
+			<geometry>
+				<mesh filename="package://mars_rover/meshes/arm_03_fixed.dae" scale="${scale_XYZ} ${scale_XYZ} ${scale_XYZ}"/>
 			</geometry>
 		</visual>
@@ -235,12 +235,12 @@
 					rpy="0 0 0"/>
 			<geometry>
-				<mesh filename="/home/spaceros-user/src/spaceros_demo/install/mars_rover/share/mars_rover/meshes/arm_04_fixed.dae" scale="${scale_XYZ} ${scale_XYZ} ${scale_XYZ}"/>
-			</geometry>
-		</collision>
-		<visual>
-			<origin xyz="0 0 0"
-					rpy="0 0 0"/>
-			<geometry>
-				<mesh filename="/home/spaceros-user/src/spaceros_demo/install/mars_rover/share/mars_rover/meshes/arm_04_fixed.dae" scale="${scale_XYZ} ${scale_XYZ} ${scale_XYZ}"/>
+				<mesh filename="package://mars_rover/meshes/arm_04_fixed.dae" scale="${scale_XYZ} ${scale_XYZ} ${scale_XYZ}"/>
+			</geometry>
+		</collision>
+		<visual>
+			<origin xyz="0 0 0"
+					rpy="0 0 0"/>
+			<geometry>
+				<mesh filename="package://mars_rover/meshes/arm_04_fixed.dae" scale="${scale_XYZ} ${scale_XYZ} ${scale_XYZ}"/>
 			</geometry>
 		</visual>
@@ -303,12 +303,12 @@
 					rpy="0 0 0"/>
 			<geometry>
-				<mesh filename="/home/spaceros-user/src/spaceros_demo/install/mars_rover/share/mars_rover/meshes/arm_tools_fixed.dae" scale="${scale_XYZ} ${scale_XYZ} ${scale_XYZ}"/>
-			</geometry>
-		</collision>
-		<visual>
-			<origin xyz="0 0 0"
-					rpy="0 0 0"/>
-			<geometry>
-				<mesh filename="/home/spaceros-user/src/spaceros_demo/install/mars_rover/share/mars_rover/meshes/arm_tools_fixed.dae" scale="${scale_XYZ} ${scale_XYZ} ${scale_XYZ}"/>
+				<mesh filename="package://mars_rover/meshes/arm_tools_fixed.dae" scale="${scale_XYZ} ${scale_XYZ} ${scale_XYZ}"/>
+			</geometry>
+		</collision>
+		<visual>
+			<origin xyz="0 0 0"
+					rpy="0 0 0"/>
+			<geometry>
+				<mesh filename="package://mars_rover/meshes/arm_tools_fixed.dae" scale="${scale_XYZ} ${scale_XYZ} ${scale_XYZ}"/>
 			</geometry>
 		</visual>

File: mars_rover/urdf/curiosity_mars_rover.xacro.urdf (robot description, URDF)
Before this commit: robot curiosity_mars_rover, 49 links, 48 joints
Links:
- link arm_01: geometry collision mesh filename=package://meshes/arm_01_fixed.dae scale=1.0 1.0 1.0; visual mesh filename=package://meshes/arm_01_fixed.dae scale=1.0 1.0 1.0
- link arm_02: geometry collision mesh filename=package://meshes/arm_01_fixed.dae scale=1.0 1.0 1.0; visual mesh filename=package://meshes/arm_02_fixed.dae scale=1.0 1.0 1.0
- link arm_03: geometry collision mesh filename=package://meshes/arm_03_fixed.dae scale=1.0 1.0 1.0; visual mesh filename=package://meshes/arm_03_fixed.dae scale=1.0 1.0 1.0
- link arm_04: geometry collision mesh filename=package://meshes/arm_04_fixed.dae scale=1.0 1.0 1.0; visual mesh filename=package://meshes/arm_04_fixed.dae scale=1.0 1.0 1.0
- link arm_tools: geometry collision mesh filename=package://meshes/arm_tools_fixed.dae scale=1.0 1.0 1.0; visual mesh filename=package://meshes/arm_tools_fixed.dae scale=1.0 1.0 1.0
- link back_wheel_L: geometry collision cylinder length=0.39473 radius=0.242647; visual mesh filename=package://meshes/wheel_fixed.dae scale=1.0 1.0 1.0
- link back_wheel_R: geometry collision cylinder length=0.39473 radius=0.242647; visual mesh filename=package://meshes/wheel_fixed.dae scale=1.0 1.0 1.0
- link chassis: geometry collision mesh scale=1.0 1.0 1.0 uri=package://meshes/chassis_full_fixed_glitch_v2.dae; visual mesh filename=package://meshes/chassis_full_fixed_glitch_v2.dae scale=1.0 1.0 1.0
- link front_wheel_L: geometry collision cylinder length=0.39473 radius=0.242647; visual mesh filename=package://meshes/wheel_fixed.dae scale=1.0 1.0 1.0
- link front_wheel_R: geometry collision cylinder length=0.39473 radius=0.242647; visual mesh filename=package://meshes/wheel_fixed.dae scale=1.0 1.0 1.0
- link left_axis: geometry collision mesh filename=package://meshes/left_axis_jointfix_v2.dae scale=1.0 1.0 1.0; visual mesh filename=package://meshes/left_axis_jointfix_v2.dae scale=1.0 1.0 1.0
- link mast_02: geometry collision mesh filename=package://meshes/mast_02_fixed.dae scale=1.0 1.0 1.0; visual mesh filename=package://meshes/mast_02_fixed.dae scale=1.0 1.0 1.0
- link mast_cameras: geometry collision mesh filename=package://meshes/mast_cameras.dae scale=1.0 1.0 1.0; visual mesh filename=package://meshes/mast_cameras.dae scale=1.0 1.0 1.0
- link mast_p: geometry collision mesh filename=package://meshes/mast_p_fixed.dae scale=1.0 1.0 1.0; visual mesh filename=package://meshes/mast_p_fixed.dae scale=1.0 1.0 1.0
- link middle_wheel_L: geometry collision cylinder length=0.39473 radius=0.242647; visual mesh filename=package://meshes/wheel_fixed.dae scale=1.0 1.0 1.0
- link middle_wheel_R: geometry collision cylinder length=0.39473 radius=0.242647; visual mesh filename=package://meshes/wheel_fixed.dae scale=1.0 1.0 1.0
- link right_axis: geometry collision mesh filename=package://meshes/right_axis_jointfix_v2.dae scale=1.0 1.0 1.0; visual mesh filename=package://meshes/right_axis_jointfix_v2.dae scale=1.0 1.0 1.0
- link suspension_arm_B2_L: geometry collision mesh filename=package://meshes/suspension_arm_B2_L_fixed.dae scale=1.0 1.0 1.0; visual mesh filename=package://meshes/suspension_arm_B2_L_fixed.dae scale=1.0 1.0 1.0
- link suspension_arm_B2_R: geometry collision mesh filename=package://meshes/suspension_arm_B2_R_fixed.dae scale=1.0 1.0 1.0; visual mesh filename=package://meshes/suspension_arm_B2_R_fixed.dae scale=1.0 1.0 1.0
- link suspension_arm_B_L: geometry collision mesh filename=package://meshes/suspension_arm_B_L_fixed.dae scale=1.0 1.0 1.0; visual mesh filename=package://meshes/suspension_arm_B_L_fixed.dae scale=1.0 1.0 1.0
- link suspension_arm_B_R: geometry collision mesh filename=package://meshes/suspension_arm_B_R_fixed.dae scale=1.0 1.0 1.0; visual mesh filename=package://meshes/suspension_arm_B_R_fixed.dae scale=1.0 1.0 1.0
- link suspension_arm_F_L: geometry collision mesh filename=package://meshes/suspension_arm_F_L_fixed.dae scale=1.0 1.0 1.0; visual mesh filename=package://meshes/suspension_arm_F_L_fixed.dae scale=1.0 1.0 1.0
- link suspension_arm_F_R: geometry collision mesh filename=package://meshes/suspension_arm_F_R_fixed.dae scale=1.0 1.0 1.0; visual mesh filename=package://meshes/suspension_arm_F_R_fixed.dae scale=1.0 1.0 1.0
- link suspension_steer_B_L: geometry collision mesh filename=package://meshes/suspension_steer_B_L_fixed.dae scale=1.0 1.0 1.0; visual mesh filename=package://meshes/suspension_steer_B_L_fixed.dae scale=1.0 1.0 1.0
- link suspension_steer_B_R: geometry collision mesh filename=package://meshes/suspension_steer_B_R_fixed.dae scale=1.0 1.0 1.0; visual mesh filename=package://meshes/suspension_steer_B_R_fixed.dae scale=1.0 1.0 1.0
- link suspension_steer_F_L: geometry collision mesh filename=package://meshes/suspension_steer_F_L_fixed.dae scale=1.0 1.0 1.0; visual mesh filename=package://meshes/suspension_steer_F_L_fixed.dae scale=1.0 1.0 1.0
- link suspension_steer_F_R: geometry collision mesh filename=package://meshes/suspension_steer_F_R_fixed.dae scale=1.0 1.0 1.0; visual mesh filename=package://meshes/suspension_steer_F_R_fixed.dae scale=1.0 1.0 1.0
